File: KiCAD/SNES-Exp-Bridge/SNES-Exp-Bridge.kicad_pcb (KiCad board)
At the start: 4 copper layers, 72 x 68 mm, 4 parts, among them J1 Conn_02x14_Odd_Even_MountingP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, J2 DB25_Socket_MountingHoles, J3 AudioJack3_Ground, J4 AudioJack3_Ground

Commit message: Add files via upload
Routing:
- net /PA0: track 55.5 -> 56.9 mm
- net /MONO_OUT: track 98.2 -> 97.5 mm
Other:
- board text added: "1 2 3 4 5 6 7 8 9 10 11 12 13"
- board text added: "14 15 15 17 18 19 20 21 22 23 24 25"
- board text added: "D3 D4 D5 D6 D7 RST 5V SMP CLK DOT CLK GND EXPAND IRQ"
- board text added: "PA0 PA1 PA2 PA3 PA4 PA5 PA6 PA7 PAWR PARD D0 D1 D2"
- board text added: "R: MONO OUT L: MONO OUT"
- board text added: "R: SR IN L: SL IN"

Commit message: Add files via upload
Parts:
- J1: footprint Connector_PinSocket_2.00mm:PinSocket_2x14_P2.00mm_Vertical_SMD -> Library:SAMTEC_MEC2-50-01-X-TH1-WT
- moved J1 2.46 mm to (171.0, 69.8), turned to 0 degrees
Routing:
- net /SL_IN: track 116.6 -> 95.5 mm
- net /D4: track 59.7 -> 52.4 mm, vias 1 -> 0
- net /D6: track 60.3 -> 53.9 mm, vias 1 -> 0
- net /rst_n: track 61.8 -> 55.4 mm, vias 1 -> 0
- net /SMP_CLK: track 63.2 -> 57.1 mm, vias 1 -> 0
- net /SR_IN: track 93.6 -> 88.8 mm
- net /MONO_OUT: track 97.5 -> 93.2 mm
- net /PA0: track 56.9 -> 53.8 mm
- net GND: track 2.90 -> 0.00 mm, vias 1 -> 0
- net /IRQ_n: track 53.6 -> 56.4 mm, vias 1 -> 0
- net /EXPAND: track 53.3 -> 56.0 mm, vias 1 -> 0
- net /PA1: track 48.4 -> 51.0 mm
- net /PA7: track 52.8 -> 55.4 mm
- net /DOT_CLK: track 51.6 -> 54.1 mm, vias 1 -> 0
- net /D5: track 47.2 -> 49.7 mm, vias 1 -> 0
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