File: KiCAD/SNES-Exp-Bridge/SNES-Exp-Bridge.kicad_sch (KiCad schematic)
At the start: 4 parts, among them J1 Conn_02x14_Odd_Even_MountingP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, J2 DB25_Socket_MountingHoles, J3 AudioJack3_Ground, J4 AudioJack3_Ground

Commit message: Add files via upload
Parts:
- J1: value Conn_02x14_Odd_Even_MountingPin -> MEC2-50-01-L-TH1; footprint Connector_PinSocket_2.00mm:PinSocket_2x14_P2.00mm_Vertical_SMD -> Library:SAMTEC_MEC2-50-01-X-TH1-WT
Changed lines of the file:
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@@
 			)
 		)
-		(property "Value" "Conn_02x14_Odd_Even_MountingPin"
+		(property "Value" "MEC2-50-01-L-TH1"
 			(at 132.08 30.48 0)
 			(effects
@@
 			)
 		)
-		(property "Footprint" "Connector_PinSocket_2.00mm:PinSocket_2x14_P2.00mm_Vertical_SMD"
+		(property "Footprint" "Library:SAMTEC_MEC2-50-01-X-TH1-WT"
 			(at 130.81 49.53 0)
 			(effects
